Commit message: add camera and tune gripper

File: urdf/poppy_ergo_jr.urdf.xacro (robot description, xacro)
@@ -1,7 +1,115 @@
 <?xml version="1.0" encoding="UTF-8"?>
 <robot xmlns:xacro="http://www.ros.org/wiki/xacro" name="poppy_ergo_jr">
+  <!-- Properties -->
+  <xacro:property name="namespace" value="ergo_jr" />
   <xacro:arg name="lamp" default="false"/>
   <xacro:arg name="gripper" default="false"/>
-  <link name="base_link">
+  <xacro:arg name="fixed" default="true"/>
+  <xacro:property name="is_fixed" value="true"/>
+  <!-- Macro to add a camera. -->
+  <xacro:macro name="camera_macro"
+    params="namespace parent_link camera_suffix frame_rate
+      horizontal_fov image_width image_height image_format min_distance
+      max_distance noise_mean noise_stddev enable_visual *cylinder *origin">
+    <link name="${namespace}/camera_${camera_suffix}_link">
+      <!-- <collision> -->
+      <!--   <origin xyz="0 0 0" rpy="0 0 0" /> -->
+      <!--   <geometry> -->
+      <!--     <xacro:insert_block name="cylinder" /> -->
+      <!--   </geometry> -->
+      <!-- </collision> -->
+      <xacro:if value="${enable_visual}">
+        <visual>
+          <origin xyz="0 0 0" rpy="0 1.57079632679 0" />
+          <geometry>
+            <xacro:insert_block name="cylinder" />
+          </geometry>
+          <material name="red">
+		     <color rgba="1 0 0 1"/>
+	  </material>
+        </visual>
+      </xacro:if>
+      <inertial>
+        <mass value="1e-5" />
+        <origin xyz="0 0 0" rpy="0 0 0" />
+        <inertia ixx="1e-6" ixy="0" ixz="0" iyy="1e-6" iyz="0" izz="1e-6" />
+      </inertial>
+    </link>
+    <joint name="${namespace}/camera_${camera_suffix}_joint" type="fixed">
+      <xacro:insert_block name="origin" />
+      <parent link="${parent_link}" />
+      <child link="${namespace}/camera_${camera_suffix}_link" />
+    </joint>
+    <gazebo reference="${namespace}/camera_${camera_suffix}_link">
+      <sensor type="camera" name="${namespace}_camera_${camera_suffix}">
+        <update_rate>${frame_rate}</update_rate>
+        <camera name="head">
+          <horizontal_fov>${horizontal_fov}</horizontal_fov>
+          <image>
+            <width>${image_width}</width>
+            <height>${image_height}</height>
+            <format>${image_format}</format>
+          </image>
+          <clip>
+            <near>${min_distance}</near>
+            <far>${max_distance}</far>
+          </clip>
+          <noise>
+            <type>gaussian</type>
+            <!-- Noise is sampled independently per pixel on each frame.
+                 That pixel's noise value is added to each of its color
+                 channels, which at that point lie in the range [0,1]. -->
+            <mean>${noise_mean}</mean>
+            <stddev>${noise_stddev}</stddev>
+          </noise>
+        </camera>
+        <plugin name="${namespace}_camera_${camera_suffix}_controller" filename="libgazebo_ros_camera.so">
+          <robotNamespace>${namespace}</robotNamespace>
+          <alwaysOn>true</alwaysOn>
+          <updateRate>${frame_rate}</updateRate>
+          <cameraName>camera_${camera_suffix}</cameraName>
+          <imageTopicName>image_raw</imageTopicName>
+          <cameraInfoTopicName>camera_info</cameraInfoTopicName>
+          <frameName>camera_${camera_suffix}_link</frameName>
+          <hackBaseline>0.0</hackBaseline>
+	  <Cx>2.0500638605704751e+02</Cx>
+	  <Cy>1.5106876398089261e+02</Cy>
+	  <focalLength>3.2390967091609349e+02</focalLength>
+          <distortionK1>1.4043219721770492e-01</distortionK1>
+          <distortionK2>-1.3210129724889583e-01</distortionK2>
+          <distortionK3>-3.6452869939025279e-01</distortionK3>
+          <distortionT1>-5.1782301614838704e-04</distortionT1>
+          <distortionT2>-5.2090817919999092e-03</distortionT2>
+        </plugin>
+      </sensor>
+    </gazebo>
+  </xacro:macro>
+<xacro:camera_macro
+    namespace="${namespace}"
+    parent_link="base_link"
+    camera_suffix="ergo"
+    frame_rate="30.0"
+    horizontal_fov="1.12825740656329"
+    image_width="800"
+    image_height="600"
+    image_format="R8G8B8"
+    min_distance="0.02"
+    max_distance="400"
+    noise_mean="0.0"
+    noise_stddev="0.001"
+    enable_visual="True"
+    >
+    <!-- <box size="0.01 0.01 0.01" /> -->
+    <cylinder length="0.01" radius="0.007" />
+    <origin xyz="0.0 -0.025 0.02" rpy="0 -0.39269908169872414 -1.57079632679"/>
+</xacro:camera_macro>
+<xacro:if value="$(arg fixed)">
+<link name="world"/>
+  <joint name="fixed" type="fixed">
+    <parent link="world"/>
+    <child link="base_link"/>
+  </joint>
+</xacro:if>
+ <link name="base_link">
     <visual>
       <origin xyz="0 0 0" rpy="0 0 0" />
@@ -14,9 +122,25 @@
     </visual>
     <collision>
-      <origin xyz="0 0.038 0.015" rpy="0 0 0" />
-      <geometry>
-        <cylinder length="0.03" radius="0.08" />
-      </geometry>
-    </collision>
+      <origin xyz="0 0.038 0.0" rpy="0 0 0" />
+      <geometry>
+        <cylinder length="0.005" radius="0.08" />
+      </geometry>
+      <surface>
+            <contact>
+              <ode>
+                <max_vel>0</max_vel>
+                <min_depth>0.01</min_depth>
+		<kp>1e15</kp>
+		<kd>1e13</kd>
+              </ode>
+            </contact>
+      </surface>
+    </collision>
+    <xacro:if value="${is_fixed == 'false'}">
+    <inertial>
+      <mass value="0.250" />
+      <inertia ixx="0.03" iyy="0.03" izz="0.03" ixy="0.0" ixz="0.0" iyz="0.0" />
+    </inertial>
+    </xacro:if>
   </link>
   <link name="long_U">
@@ -35,7 +159,17 @@
         <cylinder length="0.02" radius="0.02" />
       </geometry>
+      <surface>
+            <contact>
+              <ode>
+                <max_vel>0</max_vel>
+                <min_depth>0.01</min_depth>
+		<kp>1e15</kp>
+		<kd>1e13</kd>
+              </ode>
+            </contact>
+      </surface>
     </collision>
     <inertial>
-      <mass value="0.1" />
+      <mass value="0.05" />
       <inertia ixx="0.03" iyy="0.03" izz="0.03" ixy="0.0" ixz="0.0" iyz="0.0" />
     </inertial>
@@ -62,7 +196,17 @@
         <cylinder length="0.05" radius="0.02" />
       </geometry>
+      <surface>
+            <contact>
+              <ode>
+                <max_vel>0</max_vel>
+                <min_depth>0.01</min_depth>
+		<kp>1e15</kp>
+		<kd>1e13</kd>
+              </ode>
+            </contact>
+      </surface>
     </collision>
     <inertial>
-      <mass value="0.1" />
+      <mass value="0.05" />
       <inertia ixx="0.03" iyy="0.03" izz="0.03" ixy="0.0" ixz="0.0" iyz="0.0" />
     </inertial>
@@ -73,4 +217,5 @@
     <child link="section_1" />
     <axis xyz="0 0 -1" />
+    <dynamics damping="0.7"/>
   </joint>
   <link name="section_2">
@@ -85,11 +230,21 @@
     </visual>
     <collision>
-      <origin xyz="0.025 0 0" rpy="0 1.5707963267949 0" />
-      <geometry>
-        <cylinder length="0.05" radius="0.02" />
-      </geometry>
+      <origin xyz="0.01 0 0" rpy="0 1.5707963267949 0" />
+      <geometry>
+        <cylinder length="0.02" radius="0.02" />
+      </geometry>
+      <surface>
+            <contact>
+              <ode>
+                <max_vel>0</max_vel>
+                <min_depth>0.01</min_depth>
+		<kp>1e15</kp>
+		<kd>1e13</kd>
+              </ode>
+            </contact>
+      </surface>
     </collision>
     <inertial>
-      <mass value="0.1" />
+      <mass value="0.05" />
       <inertia ixx="0.03" iyy="0.03" izz="0.03" ixy="0.0" ixz="0.0" iyz="0.0" />
     </inertial>
@@ -100,4 +255,5 @@
     <child link="section_2" />
     <axis xyz="0 0 -1" />
+    <dynamics damping="0.7"/>
   </joint>
   <link name="section_3">
@@ -116,7 +272,17 @@
         <cylinder length="0.05" radius="0.02" />
       </geometry>
+      <surface>
+            <contact>
+              <ode>
+                <max_vel>0</max_vel>
+                <min_depth>0.01</min_depth>
+		   <kp>1e15</kp>
+		   <kd>1e13</kd>
+              </ode>
+            </contact>
+      </surface>
     </collision>
     <inertial>
-      <mass value="0.1" />
+      <mass value="0.05" />
       <inertia ixx="0.03" iyy="0.03" izz="0.03" ixy="0.0" ixz="0.0" iyz="0.0" />
     </inertial>
@@ -127,4 +293,5 @@
     <child link="section_3" />
     <axis xyz="0 0 -1" />
+    <dynamics damping="0.7"/>
   </joint>
   <link name="section_4">
@@ -146,4 +313,5 @@
       </material>
     </visual>
+    <xacro:if value="$(arg lamp)">
     <collision>
       <origin xyz="0 -0.035 0" rpy="1.5707963267949 0 0" />
@@ -153,6 +321,32 @@
       </geometry>
     </collision>
+  </xacro:if>
+      <xacro:if value="$(arg gripper)">
+    <collision>
+      <origin xyz="0 -0.035 0" rpy="1.5707963267949 0 0" />
+      <geometry>
+        <cylinder length="0.06" radius="0.02" />
+      </geometry>
+    </collision>
+    <collision>
+      <origin xyz="0.0 -0.113 0.015" rpy="0 0 0" />
+      <geometry>
+          <box size="0.03 0.03 0.005" />
+      </geometry>
+      <surface>
+            <contact>
+	       <collide_bitmask>0x01</collide_bitmask>
+              <ode>
+                <max_vel>0</max_vel>
+                <min_depth>0.01</min_depth>
+		   <kp>1e15</kp>
+		   <kd>1e13</kd>
+              </ode>
+            </contact>
+      </surface>
+    </collision>
+      </xacro:if>
     <inertial>
-      <mass value="0.1" />
+      <mass value="0.05" />
       <inertia ixx="0.03" iyy="0.03" izz="0.03" ixy="0.0" ixz="0.0" iyz="0.0" />
     </inertial>
@@ -163,4 +357,5 @@
     <child link="section_4" />
     <axis xyz="0 0 1" />
+    <dynamics damping="0.7"/>
   </joint>
   <link name="fixed_tip" />
@@ -187,11 +382,21 @@
         </material>
       </visual>
-      <collision>
-        <origin xyz="0 -0.045 0" rpy="1.5707963267949 0 0" />
-        <geometry>
-          <cylinder length="0.06" radius="0.03" />
-          <box size="0.05 0.02 0.03" />
-        </geometry>
-      </collision>
+      <!-- <collision> -->
+      <!--   <origin xyz="0 -0.045 0" rpy="1.5707963267949 0 0" /> -->
+      <!--   <geometry> -->
+      <!--     <cylinder length="0.06" radius="0.03" /> -->
+      <!--     <box size="0.05 0.02 0.03" /> -->
+      <!--   </geometry> -->
+      <!-- <surface> -->
+      <!--       <contact> -->
+      <!--         <ode> -->
+      <!--           <max_vel>0</max_vel> -->
+      <!--           <min_depth>0.01</min_depth> -->
+      <!-- 		<kp>1e15</kp> -->
+      <!-- 		<kd>1e13</kd> -->
+      <!--         </ode> -->
+      <!--       </contact> -->
+      <!-- </surface> -->
+      <!-- </collision> -->
     </xacro:if>
     <xacro:if value="$(arg gripper)">
@@ -206,15 +411,96 @@
       </visual>
       <collision>
-        <origin xyz="0 -0.04 0" rpy="-1.5707963267949 0 0" />
+        <origin xyz="-0.015 -0.055 0" rpy="-1.5707963267949 0 0" />
         <geometry>
-          <cylinder length="0.06" radius="0.02" />
+          <box size="0.005 0.03 0.03" />
+          <!-- <cylinder length="0.06" radius="0.02" /> -->
         </geometry>
+      <surface>
+            <contact>
+	       <collide_bitmask>0x01</collide_bitmask>
+              <ode>
+                <max_vel>0</max_vel>
+                <min_depth>0.01</min_depth>
+      		   <kp>1e15</kp>
+      		   <kd>1e13</kd>
+              </ode>
+            </contact>
+      </surface>
       </collision>
     </xacro:if>
     <inertial>
-      <mass value="0.1" />
+      <mass value="0.05" />
       <inertia ixx="0.03" iyy="0.03" izz="0.03" ixy="0.0" ixz="0.0" iyz="0.0" />
     </inertial>
   </link>
+  <xacro:if value="$(arg gripper)">
+    <link name="dummy_gripper_tip">
+      <visual>
+        <origin xyz="-0.015 -0.055 0" rpy="-1.5707963267949 0 0" />
+        <geometry>
+          <box size="0.001 0.001 0.001" />
+        </geometry>
+      </visual>
+      <inertial>
+      <mass value="0.001" />
+      <inertia ixx="0.03" iyy="0.03" izz="0.03" ixy="0.0" ixz="0.0" iyz="0.0" />
+    </inertial>
+      <collision>
+        <origin xyz="-0.015 -0.055 0" rpy="-1.5707963267949 0 0" />
+        <geometry>
+          <box size="0.005 0.03 0.03" />
+          <!-- <cylinder length="0.06" radius="0.02" /> -->
+        </geometry>
+      <surface>
+            <contact>
+	       <collide_bitmask>0x01</collide_bitmask>
+              <ode>
+                <max_vel>0</max_vel>
+                <min_depth>0.01</min_depth>
+      		   <kp>1e15</kp>
+      		   <kd>1e13</kd>
+              </ode>
+            </contact>
+      </surface>
+      </collision>
+    </link>
+    <!-- <joint name="dummy_spring_joint" type="prismatic"> -->
+    <!--   <parent>section_4</parent> -->
+    <!--   <child>dummy_gripper_tip</child> -->
+    <!--   <pose>0 0 0 0 0 0</pose> -->
+    <!--   <axis> -->
+    <!-- 	<limit> -->
+    <!-- 	  <lower>-0.1</lower> -->
+    <!-- 	  <upper>0.1</upper> -->
+    <!-- 	</limit> -->
+    <!-- 	<xyz>0.0 0.0 1.0</xyz> -->
+    <!-- 	<dynamics> -->
+    <!-- 	  <spring_stiffness>2500</spring_stiffness> -->
+    <!-- 	  <spring_reference>0.06</spring_reference> -->
+    <!-- 	  <damping>20.0</damping> -->
+    <!-- 	  <friction>0.75</friction> -->
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
Commit message: various fixes for the gripper

File: urdf/poppy_ergo_jr.urdf.xacro (robot description, xacro)
@@ -175,9 +175,10 @@
     </inertial>
   </link>
-  <joint name="m1" type="continuous">
+  <joint name="m1" type="revolute">
     <origin xyz="0 0 0.0327993216120967" rpy="0 0 0" />
     <parent link="base_link" />
     <child link="long_U" />
     <axis xyz="0 0 1" />
+    <limit lower="-3.1416" upper="3.1416" effort="10" velocity="3"/>
   </joint>
   <link name="section_1">
@@ -366,5 +367,6 @@
     </xacro:if>
     <xacro:if value="$(arg gripper)">
-      <origin xyz="0 -0.11 0" rpy="-1.5707963267949 0 0" />
+      <!-- <origin xyz="0 -0.11 0" rpy="-1.5707963267949 0 0" /> -->
+      <origin xyz="0 -0.11 0" rpy="0.0 -1.5707963267949 0" />
       <parent link="section_4" />
     </xacro:if>

Commit message: gripper collision

File: urdf/poppy_ergo_jr.urdf.xacro (robot description, xacro)
@@ -121,24 +121,24 @@
       </material>
     </visual>
-    <collision>
-      <origin xyz="0 0.038 0.0" rpy="0 0 0" />
-      <geometry>
-        <cylinder length="0.005" radius="0.08" />
-      </geometry>
-      <!-- <surface> -->
-      <!--       <contact> -->
-      <!--         <ode> -->
-      <!--           <max_vel>0</max_vel> -->
-      <!--           <min_depth>0.01</min_depth> -->
-      <!-- 		<kp>1e15</kp> -->
-      <!-- 		<kd>1e13</kd> -->
-      <!--         </ode> -->
-      <!--       </contact> -->
-      <!-- </surface> -->
-    </collision>
+    <!-- <collision> -->
+    <!--   <origin xyz="0 0.038 0.0" rpy="0 0 0" /> -->
+    <!--   <geometry> -->
+    <!--     <cylinder length="0.005" radius="0.08" /> -->
+    <!--   </geometry> -->
+    <!--   <!-\- <surface> -\-> -->
+    <!--   <!-\-       <contact> -\-> -->
+    <!--   <!-\-         <ode> -\-> -->
+    <!--   <!-\-           <max_vel>0</max_vel> -\-> -->
+    <!--   <!-\-           <min_depth>0.01</min_depth> -\-> -->
+    <!--   <!-\- 		<kp>1e15</kp> -\-> -->
+    <!--   <!-\- 		<kd>1e13</kd> -\-> -->
+    <!--   <!-\-         </ode> -\-> -->
+    <!--   <!-\-       </contact> -\-> -->
+    <!--   <!-\- </surface> -\-> -->
+    <!-- </collision> -->
     <xacro:if value="${is_fixed == 'false'}">
     <inertial>
-      <mass value="0.250" />
-      <inertia ixx="0.03" iyy="0.03" izz="0.03" ixy="0.0" ixz="0.0" iyz="0.0" />
+      <mass value="0.5" />
+      <inertia ixx="0.1" iyy="0.1" izz="0.1" ixy="0.0" ixz="0.0" iyz="0.0" />
     </inertial>
     </xacro:if>
@@ -171,5 +171,5 @@
     </collision>
     <inertial>
-      <mass value="0.05" />
+      <mass value="0.01" />
       <inertia ixx="0.03" iyy="0.03" izz="0.03" ixy="0.0" ixz="0.0" iyz="0.0" />
     </inertial>
@@ -180,5 +180,36 @@
     <child link="long_U" />
     <axis xyz="0 0 1" />
-    <limit lower="-3.1416" upper="3.1416" effort="10" velocity="3"/>
+    <!-- <dynamics damping="0.7"/> -->
+    <!-- <limit lower="-2.6179938779914944" upper="2.6179938779914944" effort="1" velocity="1" stiffness="1.0e6" dissipation="0"/> -->
+    <limit lower="-2.6179938779914944" upper="2.6179938779914944" effort="1" velocity="0.5"/>
+    <!-- <pose frame=''>0 0 0 0 -0 0</pose> -->
+    <!-- <axis> -->
+    <!--     <xyz>0 0 1</xyz> -->
+    <!--     <use_parent_model_frame>0</use_parent_model_frame> -->
+    <!--     <limit> -->
+    <!--       <lower>-2.6179938779914944</lower> -->
+    <!--       <upper>2.6179938779914944</upper> -->
+    <!--       <effort>-1</effort> -->
+    <!--       <velocity>-1</velocity> -->
+    <!--     </limit> -->
+    <!--     <dynamics> -->
+    <!--       <spring_reference>0</spring_reference> -->
+    <!--       <spring_stiffness>0</spring_stiffness> -->
+    <!--       <damping>0</damping> -->
+    <!-- 	  <friction>0</friction> -->
+    <!--     </dynamics> -->
+    <!-- </axis> -->
+    <physics>
+      <ode>
+        <limit>
+          <cfm>0.0</cfm>
+          <erp>0.2</erp>
+        </limit>
+	<suspension>
+          <cfm>0.0</cfm>
+          <erp>0.2</erp>
+	</suspension>
+      </ode>
+    </physics>
   </joint>
   <link name="section_1">
@@ -209,9 +240,9 @@
     </collision>
     <inertial>
-      <mass value="0.05" />
+      <mass value="0.01" />
       <inertia ixx="0.03" iyy="0.03" izz="0.03" ixy="0.0" ixz="0.0" iyz="0.0" />
     </inertial>
   </link>
-  <joint name="m2" type="continuous">
+  <joint name="m2" type="revolute">
     <origin xyz="0 0 0.0240006783879033" rpy="0 -1.5707963267949 0" />
     <parent link="long_U" />
@@ -219,4 +250,5 @@
     <axis xyz="0 0 -1" />
     <dynamics damping="0.7"/>
+    <limit lower="-1.5707963267948966" upper="2.181661564992912" effort="1" velocity="1"/>
   </joint>
   <link name="section_2">
@@ -247,9 +279,9 @@
     </collision>
     <inertial>
-      <mass value="0.05" />
+      <mass value="0.01" />
       <inertia ixx="0.03" iyy="0.03" izz="0.03" ixy="0.0" ixz="0.0" iyz="0.0" />
     </inertial>
   </link>
-  <joint name="m3" type="continuous">
+  <joint name="m3" type="revolute">
     <origin xyz="0.054 0 0" rpy="0 0 0" />
     <parent link="section_1" />
@@ -257,4 +289,5 @@
     <axis xyz="0 0 -1" />
     <dynamics damping="0.7"/>
+    <limit lower="-1.5707963267948966" upper="1.5707963267948966" effort="1" velocity="1"/>
   </joint>
   <link name="section_3">
@@ -285,9 +318,9 @@
     </collision>
     <inertial>
-      <mass value="0.05" />
+      <mass value="0.01" />
       <inertia ixx="0.03" iyy="0.03" izz="0.03" ixy="0.0" ixz="0.0" iyz="0.0" />
     </inertial>
   </link>
-  <joint name="m4" type="continuous">
+  <joint name="m4" type="revolute">
     <origin xyz="0.045 0 0" rpy="0 -1.5707963267949 0" />
     <parent link="section_2" />
@@ -295,4 +328,5 @@
     <axis xyz="0 0 -1" />
     <dynamics damping="0.7"/>
+    <limit lower="-2.6179938779914944" upper="2.6179938779914944" effort="1" velocity="1"/>
   </joint>
   <link name="section_4">
@@ -333,5 +367,5 @@
       <origin xyz="0.0 -0.113 0.015" rpy="0 0 0" />
       <geometry>
-          <box size="0.03 0.03 0.005" />
+          <box size="0.04 0.03 0.005" />
       </geometry>
       <surface>
@@ -349,9 +383,9 @@
       </xacro:if>
     <inertial>
-      <mass value="0.05" />
+      <mass value="0.01" />
       <inertia ixx="0.03" iyy="0.03" izz="0.03" ixy="0.0" ixz="0.0" iyz="0.0" />
     </inertial>
   </link>
-  <joint name="m5" type="continuous">
+  <joint name="m5" type="revolute">
     <origin xyz="0 -0.048 0" rpy="0 -1.5707963267949 0" />
     <parent link="section_3" />
@@ -359,4 +393,5 @@
     <axis xyz="0 0 1" />
     <dynamics damping="0.7"/>
+    <limit lower="-1.5707963267948966" upper="1.5707963267948966" effort="1" velocity="1"/>
   </joint>
   <link name="fixed_tip" />
@@ -415,5 +450,5 @@
         <origin xyz="-0.015 -0.055 0" rpy="-1.5707963267949 0 0" />
         <geometry>
-          <box size="0.005 0.03 0.03" />
+          <box size="0.005 0.04 0.03" />
           <!-- <cylinder length="0.06" radius="0.02" /> -->
         </geometry>
@@ -432,5 +467,5 @@
     </xacro:if>
     <inertial>
-      <mass value="0.05" />
+      <mass value="0.01" />
       <inertia ixx="0.03" iyy="0.03" izz="0.03" ixy="0.0" ixz="0.0" iyz="0.0" />
     </inertial>
@@ -451,5 +486,5 @@
         <origin xyz="-0.015 -0.055 0" rpy="-1.5707963267949 0 0" />
         <geometry>
-          <box size="0.005 0.03 0.03" />
+          <box size="0.005 0.04 0.03" />
           <!-- <cylinder length="0.06" radius="0.02" /> -->
         </geometry>
@@ -505,5 +540,5 @@
   </joint>
   </xacro:if>
-  <joint name="m6" type="continuous">
+  <joint name="m6" type="revolute">
     <xacro:if value="$(arg lamp)">
       <origin xyz="0 -0.054 0" rpy="0 0 0" />
@@ -517,4 +552,5 @@
     <child link="section_5" />
     <dynamics damping="0.7"/>
+    <limit lower="-1.9198621771937625" upper="1.5707963267948966" effort="1" velocity="1"/>
   </joint>
   <xacro:if value="$(arg gripper)">

Commit message: fix broken meshs

File: urdf/poppy_ergo_jr.urdf.xacro (robot description, xacro)
@@ -117,7 +117,7 @@
         <mesh filename="package://poppy_ergo_jr_description/meshes/base.dae" />
       </geometry>
-      <material name="">
-        <color rgba="0.752941176470588 0.752941176470588 0.752941176470588 1" />
-      </material>
+      <!-- <material name=""> -->
+      <!--   <color rgba="0.752941176470588 0.752941176470588 0.752941176470588 1" /> -->
+      <!-- </material> -->
     </visual>
     <!-- <collision> -->
@@ -344,7 +344,7 @@
         </geometry>
       </xacro:if>
-      <material name="">
-        <color rgba="0.752941176470588 0.752941176470588 0.752941176470588 1" />
-      </material>
+      <!-- <material name=""> -->
+      <!--   <color rgba="0.752941176470588 0.752941176470588 0.752941176470588 1" /> -->
+      <!-- </material> -->
     </visual>
     <xacro:if value="$(arg lamp)">

Commit message: m6 limit for both eef

File: urdf/poppy_ergo_jr.urdf.xacro (robot description, xacro)
@@ -226,5 +226,4 @@
       <origin xyz="0 -0.054 0" rpy="0 0 0" />
       <axis xyz="0 0 1" />
-      <limit lower="-0.61" upper="0.5" effort="1" velocity="0.5"/>
     </xacro:if>
     <xacro:if value="$(arg gripper)">
@@ -232,4 +231,5 @@
       <axis xyz="0 0 -1" />
     </xacro:if>
+    <limit lower="-0.61" upper="0.5" effort="1" velocity="0.5"/>
     <parent link="section_4" />
     <child link="section_5" />
