Commit message: Cleaned per-motor limits from pypot in xacro

File: urdf/poppy_ergo_jr.urdf.xacro (robot description, xacro)
@@ -74,5 +74,5 @@
     <child link="section_1" />
     <axis xyz="0 0 -1" />
-    <limit lower="-0.5" upper="0.7" effort="1" velocity="0.5"/>
+    <limit lower="-0.84" upper="0.84" effort="1" velocity="0.5"/>
   </joint>
   <link name="section_2">
@@ -102,5 +102,5 @@
     <child link="section_2" />
     <axis xyz="0 0 -1" />
-    <limit lower="-0.5" upper="0.5" effort="1" velocity="0.5"/>
+    <limit lower="-0.84" upper="0.84" effort="1" velocity="0.5"/>
   </joint>
   <link name="section_3">
@@ -167,5 +167,5 @@
     <child link="section_4" />
     <axis xyz="0 0 1" />
-    <limit lower="-0.5" upper="0.5" effort="1" velocity="0.5"/>
+    <limit lower="-0.84" upper="0.84" effort="1" velocity="0.5"/>
   </joint>
   <link name="fixed_tip" />
@@ -231,5 +231,5 @@
       <axis xyz="0 0 -1" />
     </xacro:if>
-    <limit lower="-0.61" upper="0.5" effort="1" velocity="0.5"/>
+    <limit lower="-0.84" upper="0.84" effort="1" velocity="0.5"/>
     <parent link="section_4" />
     <child link="section_5" />

Commit message: Always add inertia term for gazebo

File: urdf/poppy_ergo_jr.urdf.xacro (robot description, xacro)
@@ -137,10 +137,10 @@
     <!--   <!-\- </surface> -\-> -->
     <!-- </collision> -->
-    <xacro:if value="${is_fixed == 'false'}">
+    <!-- <xacro:if value="${is_fixed == 'false'}"> -->
     <inertial>
       <mass value="0.5" />
       <inertia ixx="0.1" iyy="0.1" izz="0.1" ixy="0.0" ixz="0.0" iyz="0.0" />
     </inertial>
-    </xacro:if>
+    <!-- </xacro:if> -->
   </link>
   <link name="long_U">
@@ -367,5 +367,5 @@
       <origin xyz="0.0 -0.113 0.015" rpy="0 0 0" />
       <geometry>
-          <box size="0.04 0.03 0.005" />
+          <box size="0.025 0.03 0.005" />
       </geometry>
       <surface>
@@ -450,5 +450,5 @@
         <origin xyz="-0.015 -0.055 0" rpy="-1.5707963267949 0 0" />
         <geometry>
-          <box size="0.005 0.04 0.03" />
+          <box size="0.005 0.025 0.03" />
           <!-- <cylinder length="0.06" radius="0.02" /> -->
         </geometry>
@@ -486,5 +486,5 @@
         <origin xyz="-0.015 -0.055 0" rpy="-1.5707963267949 0 0" />
         <geometry>
-          <box size="0.005 0.04 0.03" />
+          <box size="0.005 0.025 0.03" />
           <!-- <cylinder length="0.06" radius="0.02" /> -->
         </geometry>
@@ -531,6 +531,6 @@
     <!--   </physics> -->
     <!-- </joint> -->
-  <joint name="dummy_fixed" type="prismatic">
-  <!-- <joint name="dummy_fixed" type="fixed"> -->
+  <joint name="dummy_fixed" type="fixed">
+  <!-- <joint name="" type="fixed"> -->
       <!-- <origin xyz="0 0 0" rpy="0 0 0" /> -->
       <parent link="section_5" />
@@ -634,5 +634,5 @@
       <contact>
         <ode>
-	  <min_depth>0.003</min_depth>
+	  <min_depth>0.001</min_depth>
 	  <max_vel>0</max_vel>
         </ode>
@@ -657,5 +657,5 @@
       <contact>
         <ode>
-	  <min_depth>0.003</min_depth>
+	  <min_depth>0.001</min_depth>
 	  <max_vel>0</max_vel>
         </ode>
