Commit message: Drop unsupported inertia

File: urdf/poppy_ergo_jr.urdf (robot description, URDF)
Before this commit: robot PoppyErgoJr, 7 links, 6 joints
Links:
- link base_link: mass 0.0802410895423366 -> None

Commit message: Axis direction updated

File: urdf/poppy_ergo_jr.urdf (robot description, URDF)
Before this commit: robot PoppyErgoJr, 7 links, 6 joints
Joints:
- joint m1: axis 0 0 -1 -> 0 0 1
- joint m2: axis -1 0 0 -> 1 0 0
- joint m3: axis -1 0 0 -> 1 0 0
- joint m5: axis -1 0 0 -> 1 0 0

Commit message: Fix joints in order to defaults

File: urdf/poppy_ergo_jr.urdf (robot description, URDF)
Before this commit: robot PoppyErgoJr, 7 links, 6 joints
Joints:
- joint m1: origin xyz=0 0 0.0327993216120967 rpy=-6.12303176911189E-17 0 0 -> xyz=0 0 0.0327993216120967 rpy=0 0 0
- joint m2: axis 1 0 0 -> 0 0 -1; origin xyz=0 0 0.0240006783879033 rpy=1.5707963267949 0 0 -> xyz=0 0 0.0240006783879033 rpy=0 -1.5707963267949 0
- joint m3: axis 1 0 0 -> 0 0 -1; origin xyz=0 0 0.054 rpy=0 0 0 -> xyz=0.054 0 0 rpy=0 0 0
- joint m4: axis 0 0 1 -> 0 0 -1; origin xyz=0 0 0.045 rpy=0 0 3.14159265358979 -> xyz=0.045 0 0 rpy=0 -1.5707963267949 0
- joint m5: axis 1 0 0 -> 0 0 1; origin xyz=0 -0.048 0 rpy=-1.5707963267949 0 0 -> xyz=0 -0.048 0 rpy=0 -1.5707963267949 0
- joint m6: origin xyz=0 -0.058 0 rpy=0 0 0 -> xyz=0 -0.058 0 rpy=0 -1.5707963267949 0

Commit message: Cleaned outdated inertias + updated collisions

File: urdf/poppy_ergo_jr.urdf (robot description, URDF)
Before this commit: robot PoppyErgoJr, 7 links, 6 joints
Links:
- link long_U: mass 0.0042118228619085 -> None
- link section_1: mass 0.0201321844066136 -> None
- link section_2: mass 0.017821725151696 -> None
- link section_3: mass 0.0201321844066136 -> None
- link section_4: mass 0.0201321844066137 -> None
- link tip: mass 0.0164859649700598 -> None

Commit message: Added the collision model

File: urdf/poppy_ergo_jr.urdf (robot description, URDF)
Before this commit: robot PoppyErgoJr, 7 links, 6 joints
Links:
- link base_link: geometry collision cylinder length=0.03 radius=0.08; visual mesh filename=package://poppy_ergo_jr_description/meshes/base.dae
- link long_U: geometry collision cylinder length=0.02 radius=0.02; visual mesh filename=package://poppy_ergo_jr_description/meshes/long_U.dae
- link section_1: geometry collision cylinder length=0.05 radius=0.02; visual mesh filename=package://poppy_ergo_jr_description/meshes/section_1.dae
- link section_2: geometry collision cylinder length=0.05 radius=0.02; visual mesh filename=package://poppy_ergo_jr_description/meshes/section_2.dae
- link section_3: geometry collision cylinder length=0.05 radius=0.02; visual mesh filename=package://poppy_ergo_jr_description/meshes/section_3.dae
- link section_4: geometry collision cylinder length=0.06 radius=0.02; visual mesh filename=package://poppy_ergo_jr_description/meshes/section_4.dae
- link tip: geometry collision cylinder length=0.06 radius=0.02; visual mesh filename=package://poppy_ergo_jr_description/meshes/gripper.dae

Commit message: URDF Update for Gazebo
Update from Moveit setup assistant

File: urdf/poppy_ergo_jr.urdf (robot description, URDF)
Before this commit: robot PoppyErgoJr, 7 links, 6 joints
Links:
- link base_link: mass None -> 0.1
- link long_U: mass None -> 0.1
- link section_1: mass None -> 0.1
- link section_2: mass None -> 0.1
- link section_3: mass None -> 0.1
- link section_4: mass None -> 0.1
- link tip: mass None -> 0.1

Commit message: Add fixed_tip and moving_tip to URDF

File: urdf/poppy_ergo_jr.urdf (robot description, URDF)
Before this commit: robot poppy_ergo_jr, 7 links, 6 joints
Links:
- removed link tip
- added link fixed_tip
- added link moving_tip
- added link section_5, mass 0.1; collision cylinder length=0.06 radius=0.02; visual mesh filename=package://poppy_ergo_jr_description/meshes/gripper.dae
Joints:
- added joint t7f: type fixed, parent section_4, child fixed_tip, origin xyz=0 -0.11 0 rpy=-1.5707963267949 0 0
- added joint t7m: type fixed, parent section_5, child moving_tip, origin xyz=0 -0.052 0 rpy=-1.5707963267949 0 0
- joint m6: child tip -> section_5

Commit message: Return m6 joint

File: urdf/poppy_ergo_jr.urdf (robot description, URDF)
Before this commit: robot poppy_ergo_jr, 9 links, 8 joints
Joints:
- joint m6: axis 0 0 1 -> 0 0 -1

Commit message: Integrated the lamp with Xacro

File: urdf/poppy_ergo_jr.urdf (robot description, URDF)
Before this commit: robot poppy_ergo_jr, 9 links, 8 joints
Links:
- removed link moving_tip
- link section_4: geometry collision cylinder length=0.06 radius=0.02; visual mesh filename=package://poppy_ergo_jr_description/meshes/section_1.dae
- link section_5: geometry collision cylinder length=0.06 radius=0.03; visual mesh filename=package://poppy_ergo_jr_description/meshes/lamp.dae
Joints:
- removed joint t7m
- joint m6: axis 0 0 -1 -> 0 0 1; origin xyz=0 -0.058 0 rpy=0 -1.5707963267949 0 -> xyz=0 -0.054 0 rpy=0 0 0
- joint t7f: origin xyz=0 -0.11 0 rpy=-1.5707963267949 0 0 -> xyz=0 -0.075 0 rpy=-1.5707963267949 0 0; parent section_4 -> section_5

Commit message: clean urdf

File: urdf/poppy_ergo_jr.urdf (robot description, URDF)
Before this commit: robot poppy_ergo_jr, 8 links, 7 joints
Links:
- added link dummy_gripper_tip, mass 0.001; collision box size=0.005 0.04 0.03; visual box size=0.001 0.001 0.001
- added link ergo_jr/camera_ergo_link, mass 1e-5; visual cylinder length=0.01 radius=0.007
- added link moving_tip
- added link world
- link base_link: geometry visual mesh filename=package://poppy_ergo_jr_description/meshes/base.dae
- link long_U: mass 0.1 -> 0.01
- link section_1: mass 0.1 -> 0.01
- link section_2: mass 0.1 -> 0.01; geometry collision cylinder length=0.02 radius=0.02; visual mesh filename=package://poppy_ergo_jr_description/meshes/section_2.dae
- link section_3: mass 0.1 -> 0.01
- link section_4: mass 0.1 -> 0.01; geometry collision box size=0.04 0.03 0.005; collision cylinder length=0.06 radius=0.02
- link section_5: mass 0.1 -> 0.01; geometry collision box size=0.005 0.04 0.03; visual mesh filename=package://poppy_ergo_jr_description/meshes/gripper.dae
Joints:
- added joint dummy_fixed: type prismatic, parent section_5, child dummy_gripper_tip, axis 0 0 1, limit lower=0 upper=0 effort=1000 velocity=0.0
- added joint ergo_jr/camera_ergo_joint: type fixed, parent base_link, child ergo_jr/camera_ergo_link, origin xyz=0.0 -0.025 0.02 rpy=0 -0.39269908169872414 -1.57079632679
- added joint fixed: type fixed, parent world, child base_link
- added joint t7m: type fixed, parent section_5, child moving_tip, origin xyz=0 -0.052 0 rpy=-1.5707963267949 0 0
- joint m1: limit (none) -> lower=-2.6179938779914944 upper=2.6179938779914944 effort=1 velocity=0.5; type continuous -> revolute
- joint m2: limit (none) -> lower=-1.5707963267948966 upper=2.181661564992912 effort=1 velocity=1; type continuous -> revolute
- joint m3: limit (none) -> lower=-1.5707963267948966 upper=1.5707963267948966 effort=1 velocity=1; type continuous -> revolute
- joint m4: limit (none) -> lower=-2.6179938779914944 upper=2.6179938779914944 effort=1 velocity=1; type continuous -> revolute
- joint m5: limit (none) -> lower=-1.5707963267948966 upper=1.5707963267948966 effort=1 velocity=1; type continuous -> revolute
- joint m6: axis 0 0 1 -> 0 0 -1; limit (none) -> lower=-1.9198621771937625 upper=1.5707963267948966 effort=1 velocity=1; origin xyz=0 -0.054 0 rpy=0 0 0 -> xyz=0 -0.058 0 rpy=0 -1.5707963267949 0; type continuous -> revolute
- joint t7f: origin xyz=0 -0.075 0 rpy=-1.5707963267949 0 0 -> xyz=0 -0.11 0 rpy=0.0 -1.5707963267949 0; parent section_5 -> section_4

File: urdf/poppy_ergo_jr.urdf.xacro (robot description, xacro)
@@ -4,5 +4,5 @@
   <xacro:property name="namespace" value="ergo_jr" />
   <xacro:arg name="lamp" default="false"/>
-  <xacro:arg name="gripper" default="false"/>
+  <xacro:arg name="gripper" default="true"/>
   <xacro:arg name="fixed" default="true"/>
   <xacro:property name="is_fixed" value="true"/>

Commit message: URDF joints revolute with limits

File: urdf/poppy_ergo_jr.urdf (robot description, URDF)
Before this commit: robot poppy_ergo_jr, 8 links, 7 joints
Joints:
- joint m1: limit (none) -> lower=-0.84 upper=0.84 effort=1 velocity=0.5; type continuous -> revolute
- joint m2: limit (none) -> lower=-0.5 upper=0.7 effort=1 velocity=0.5; type continuous -> revolute
- joint m3: limit (none) -> lower=-0.5 upper=0.5 effort=1 velocity=0.5; type continuous -> revolute
- joint m4: limit (none) -> lower=-0.84 upper=0.84 effort=1 velocity=0.5; type continuous -> revolute
- joint m5: limit (none) -> lower=-0.5 upper=0.5 effort=1 velocity=0.5; type continuous -> revolute
- joint m6: limit (none) -> lower=-0.61 upper=0.5 effort=1 velocity=0.5; type continuous -> revolute

File: urdf/poppy_ergo_jr.urdf.xacro (robot description, xacro)
@@ -41,9 +41,10 @@
     </inertial>
   </link>
-  <joint name="m1" type="continuous">
+  <joint name="m1" type="revolute">
     <origin xyz="0 0 0.0327993216120967" rpy="0 0 0" />
     <parent link="base_link" />
     <child link="long_U" />
     <axis xyz="0 0 1" />
+    <limit lower="-0.84" upper="0.84" effort="1" velocity="0.5"/>
   </joint>
   <link name="section_1">
@@ -68,9 +69,10 @@
     </inertial>
   </link>
-  <joint name="m2" type="continuous">
+  <joint name="m2" type="revolute">
     <origin xyz="0 0 0.0240006783879033" rpy="0 -1.5707963267949 0" />
     <parent link="long_U" />
     <child link="section_1" />
     <axis xyz="0 0 -1" />
+    <limit lower="-0.5" upper="0.7" effort="1" velocity="0.5"/>
   </joint>
   <link name="section_2">
@@ -95,9 +97,10 @@
     </inertial>
   </link>
-  <joint name="m3" type="continuous">
+  <joint name="m3" type="revolute">
     <origin xyz="0.054 0 0" rpy="0 0 0" />
     <parent link="section_1" />
     <child link="section_2" />
     <axis xyz="0 0 -1" />
+    <limit lower="-0.5" upper="0.5" effort="1" velocity="0.5"/>
   </joint>
   <link name="section_3">
@@ -122,9 +125,10 @@
     </inertial>
   </link>
-  <joint name="m4" type="continuous">
+  <joint name="m4" type="revolute">
     <origin xyz="0.045 0 0" rpy="0 -1.5707963267949 0" />
     <parent link="section_2" />
     <child link="section_3" />
     <axis xyz="0 0 -1" />
+    <limit lower="-0.84" upper="0.84" effort="1" velocity="0.5"/>
   </joint>
   <link name="section_4">
@@ -158,9 +162,10 @@
     </inertial>
   </link>
-  <joint name="m5" type="continuous">
+  <joint name="m5" type="revolute">
     <origin xyz="0 -0.048 0" rpy="0 -1.5707963267949 0" />
     <parent link="section_3" />
     <child link="section_4" />
     <axis xyz="0 0 1" />
+    <limit lower="-0.5" upper="0.5" effort="1" velocity="0.5"/>
   </joint>
   <link name="fixed_tip" />
@@ -217,8 +222,9 @@
     </inertial>
   </link>
-  <joint name="m6" type="continuous">
+  <joint name="m6" type="revolute">
     <xacro:if value="$(arg lamp)">
       <origin xyz="0 -0.054 0" rpy="0 0 0" />
       <axis xyz="0 0 1" />
+      <limit lower="-0.61" upper="0.5" effort="1" velocity="0.5"/>
     </xacro:if>
     <xacro:if value="$(arg gripper)">

Commit message: Cleaned per-motor limits from pypot

File: urdf/poppy_ergo_jr.urdf (robot description, URDF)
Before this commit: robot poppy_ergo_jr, 8 links, 7 joints
Joints:
- joint m2: limit lower=-0.5 upper=0.7 effort=1 velocity=0.5 -> lower=-0.84 upper=0.84 effort=1 velocity=0.5
- joint m3: limit lower=-0.5 upper=0.5 effort=1 velocity=0.5 -> lower=-0.84 upper=0.84 effort=1 velocity=0.5
- joint m5: limit lower=-0.5 upper=0.5 effort=1 velocity=0.5 -> lower=-0.84 upper=0.84 effort=1 velocity=0.5
- joint m6: limit lower=-0.61 upper=0.5 effort=1 velocity=0.5 -> lower=-0.84 upper=0.84 effort=1 velocity=0.5

Commit message: Modified gripper collisions

File: urdf/poppy_ergo_jr.urdf (robot description, URDF)
Before this commit: robot poppy_ergo_jr, 12 links, 11 joints
Joints:
- joint ergo_jr/camera_ergo_joint: origin xyz=0.0 -0.025 0.02 rpy=0 -0.39269908169872414 -1.57079632679 -> xyz=0.0 -0.025 0.02 rpy=0 0 -1.57079632679

File: urdf/poppy_ergo_jr.urdf.xacro (robot description, xacro)
@@ -102,5 +102,5 @@
     <!-- <box size="0.01 0.01 0.01" /> -->
     <cylinder length="0.01" radius="0.007" />
-    <origin xyz="0.0 -0.025 0.02" rpy="0 -0.39269908169872414 -1.57079632679"/>
+    <origin xyz="0.0 -0.025 0.02" rpy="0 -0.29269908169872414 -1.57079632679"/>
 </xacro:camera_macro>
 <xacro:if value="$(arg fixed)">
